File: __Project__/hardware/Interface-Tree.kicad_sch (KiCad schematic)
At the start: 0 parts

Commit message: Update project template
Other:
- company: (none) -> ${COMPANY}
Changed lines of the file:
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@@
 	(generator_version "9.0")
 	(paper "A3")
+	(title_block
+		(date "2025-06-05")
+		(rev "${REVISION}")
+		(company "${COMPANY}")
+	)
 	(image
 		(at 215.9 135.89)

Commit message: Fix JST footprints
Other:
- title: (none) -> Interface - Tree
Changed lines of the file:
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@@
 	(paper "A3")
 	(title_block
+		(title "Interface - Tree")
 		(date "2025-06-05")
 		(rev "${REVISION}")
 		(company "${COMPANY}")
 	)
+	(text_box "[${#}] ${TITLE}"
+		(exclude_from_sim no)
+		(at 12.7 12.7 0)
+		(size 394.97 20.32)
+		(margins 5.9999 5.9999 5.9999 5.9999)
+		(stroke
+			(width -0.0001)
+			(type default)
+		)
+		(fill
+			(type none)
+		)
+		(effects
+			(font
+				(face "Times New Roman")
+				(size 8 8)
+				(thickness 1.2)
+				(bold yes)
+				(color 162 22 34 1)
+			)
+		)
+	)
 	(image
