File: Design-Blocks/Buck-Converter.kicad_blocks/ST1S14PHR_3V3_3A.kicad_block/ST1S14PHR_3V3_3A.kicad_pcb (KiCad board)
At the start: 4 copper layers, 19 parts, among them IC1501 ST1S14PHR

Commit message: Update design blocks
Parts:
- removed C1501, C1502: 10u, Capacitor_SMD:C_0805_2012Metric
- removed C1503, C1505, C1508: 100n, Capacitor_SMD:C_0402_1005Metric
- removed C1504: 68n, Capacitor_SMD:C_0402_1005Metric
- removed C1506: 150p, Capacitor_SMD:C_0402_1005Metric
- removed C1507: 470u, Capacitor_SMD:CP_Elec_6.3x7.7
- removed C1510: 33p, Capacitor_SMD:C_0402_1005Metric
- removed D1501: STPS3L60U, Diode_SMD:D_SMB
- removed IC1501: ST1S14PHR, Package_SO:HSOP-8-1EP_3.9x4.9mm_P1.27mm_EP2.41x3.1mm
- removed L1501: 10u, Inductor_SMD:L_Wuerth_HCI-7050
- removed R1501, R1502: 100k, Resistor_SMD:R_0402_1005Metric
- removed R1504: 82k5, Resistor_SMD:R_0402_1005Metric
- removed R1505: 48k7, Resistor_SMD:R_0402_1005Metric
- removed TP1501, TP1502, TP1504: ~, Testpoints_Kampi:TestPoint_Pad_1.0x1.0mm
- added C901: 10u, Capacitor_SMD:C_0805_2012Metric, F.Cu at (108.5, 164.5)
- added C902: 10u, Capacitor_SMD:C_0805_2012Metric, F.Cu at (108.5, 166.6)
- added C903: 100n, Capacitor_SMD:C_0402_1005Metric, F.Cu at (108.4, 168.1)
- added C904: 68n, Capacitor_SMD:C_0402_1005Metric, F.Cu at (108.4, 169.0)
- added C905: 100n, Capacitor_SMD:C_0402_1005Metric, F.Cu at (105.2, 172.1)
- added C906: 150p, Capacitor_SMD:C_0402_1005Metric, F.Cu at (111.3, 178.2)
- added C907: 470u, Capacitor_SMD:CP_Elec_6.3x7.7, F.Cu at (100.5, 185.1)
- added C908: 100n, Capacitor_SMD:C_0402_1005Metric, F.Cu at (100.3, 189.2)
- added C909: 33p, Capacitor_SMD:C_0402_1005Metric, F.Cu at (100.3, 190.2)
- added D901: STPS3L60U, Diode_SMD:D_SMB, F.Cu at (100.9, 170.8)
- added IC901: ST1S14PHR, Package_SO:HSOP-8-1EP_3.9x4.9mm_P1.27mm_EP2.41x3.1mm, F.Cu at (108.5, 173.3)
- added L901: 10u, Inductor_SMD:L_Wuerth_HCI-7050, F.Cu at (101.8, 177.2)
- added LED901: Power Good, LED_SMD:LED_0805_2012Metric, F.Cu at (113.6, 179.7)
- added R901: 100k, Resistor_SMD:R_0402_1005Metric, F.Cu at (112.2, 170.7)
- added R902: 100k, Resistor_SMD:R_0402_1005Metric, F.Cu at (109.1, 178.1)
- added R904: 150R, Resistor_SMD:R_0402_1005Metric, F.Cu at (110.6, 179.7)
- added R905: 82k5, Resistor_SMD:R_0402_1005Metric, F.Cu at (110.4, 178.2)
- added R906: 48k7, Resistor_SMD:R_0402_1005Metric, F.Cu at (111.8, 174.9)
- added TP901: ~, Testpoints_Kampi:TestPoint_Pad_1.0x1.0mm, F.Cu at (105.6, 164.5)
- added TP903: ~, Testpoints_Kampi:TestPoint_Pad_1.0x1.0mm, F.Cu at (112.9, 177.6)
- added TP904: ~, Testpoints_Kampi:TestPoint_Pad_1.0x1.0mm, F.Cu at (105.3, 182.6)
Routing:
- net Net-(IC901-PG): track 0.00 -> 9.15 mm, vias 0 -> 2
- net Net-(IC901-BOOT): track 0.00 -> 3.98 mm
- net Net-(IC1501-BOOT): track 2.89 -> 0.00 mm
- net Net-(IC901-~{EN1}): track 0.00 -> 1.59 mm
- net Net-(IC1501-~{EN1}): track 1.59 -> 0.00 mm
- net Net-(LED901-A): track 0.00 -> 1.55 mm
- net /Project Architecture/PCIe/SSD-Power: track 1.35 -> 0.00 mm
- net /Project Architecture/Modem/Modem-Power: track 0.00 -> 1.35 mm
- net /Project Architecture/PCIe/V_{SSD}: track 1.01 -> 0.00 mm
- net /Project Architecture/Modem/V_{Modem}: track 0.00 -> 1.01 mm
- net GND: vias 11 -> 33
- added copper zone on F.Cu, net /Project Architecture/Modem/V_{Modem}
- added copper zone on F.Cu, net Net-(D901-K)
- added copper zone on F.Cu, net Net-(IC901-FB)
- removed copper zone on F.Cu, net /Project Architecture/PCIe/V_{SSD}
- removed copper zone on F.Cu, net Net-(D1501-K)
- removed copper zone on F.Cu, net Net-(IC1501-FB)
